File: inputs.kicad_sch (KiCad schematic)
At the start: 50 parts, among them J4 CV Input 1, J5 CV Input 2, J6 CV Input 3, J7 CV Input 4, P1 B10K, P2 B10K, P3 B10K, P4 B10K, U1 TL074, U2 TL074

Commit message: reorder annotations, replot pdf schematic
Parts:
- renumbered C11 to C12, C12 to C13, C13 to C14, C14 to C15, C15 to C16, C16 to C17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
